Commit message: better

File: src/mirmi_robot_description/urdf/robot.urdf (robot description, URDF)
Before this commit: robot mirmi_robot, 9 links, 8 joints
Links:
- removed link dock_tag
- removed link map
- removed link vicon/Robot_1/Robot_1
- removed link vicon/Tag_0/Tag_0
- removed link vicon/world
- removed link vicon_real_target
- removed link world
- added link camera_link
- added link gps_link
- added link imu_link
- added link lidar_link
Joints:
- removed joint base_link_to_camera
- removed joint map_to_world
- removed joint vicon_robot_to_base_link
- removed joint vicon_tag_to_dock_tag
- removed joint vicon_tag_to_real_target
- removed joint vicon_world_to_robot_1
- removed joint vicon_world_to_tag_0
- removed joint world_to_vicon_world
- added joint base_link_to_camera_link: type fixed, parent base_link, child camera_link, origin xyz=0.1875 0.0 -0.1875 rpy=0.0 0.0 0.0
- added joint base_link_to_gps: type fixed, parent base_link, child gps_link, origin xyz=0.0 0.0 0.20 rpy=0.0 0.0 0.0
- added joint base_link_to_imu: type fixed, parent base_link, child imu_link, origin xyz=0.0 0.0 0.0 rpy=0.0 0.0 0.0
- added joint base_link_to_lidar: type fixed, parent base_link, child lidar_link, origin xyz=0.05 0.0 0.15 rpy=0.0 0.0 0.0
- added joint camera_link_to_optical: type fixed, parent camera_link, child camera_color_optical_frame, origin xyz=0.0 0.0 0.0 rpy=1.5707963267948966 0.0 1.5707963267948966

Commit message: added pole detector

File: src/mirmi_robot_description/urdf/robot.urdf (robot description, URDF)
Before this commit: robot mirmi_robot, 6 links, 5 joints
Links:
- removed link gps_link
- removed link imu_link
- removed link lidar_link
Joints:
- removed joint base_link_to_gps
- removed joint base_link_to_imu
- removed joint base_link_to_lidar
